File: pcb/Radio_bridge.brd (EAGLE design)
At the start: 70 x 110 mm, 45 parts, among them IC1 LM833D, J1 SJ-2509N, J2 SJ1-3523N, J4 G-1005B, SW1 EVQ-PF008K, SW2 EVQ-PF008K, U1 ESP32-DEVKITC-32D, U3 LMV7219M5X

Commit message: Rev2 PCB fixes
Parts:
- added C12: 100uF, ruark2:1210
- moved JP2 21.8 mm to (18.0, 85.6)
- moved JP4 21.8 mm to (39.9, 85.6)
Connections:
- new net N$11: C12.2, R16.3
- net GND: now also C12.1; no longer R16.3
- net MOSI: now also U1.J3-2; no longer U1.J2-11
- net N$4: now also U1.J3-11; no longer U1.J3-15
- net SCK: now also U1.J3-9; no longer U1.J3-10
- net SS: now also U1.J3-10; no longer U1.J3-9
Routing:
- net DIO0: track 68.4 -> 118.0 mm, vias 1 -> 0
- net +3V3: track 172.9 -> 126.3 mm, vias 8 -> 4
- net DIO1: track 49.0 -> 90.5 mm
- net DIO2: track 43.5 -> 84.3 mm
- net SS: track 67.0 -> 87.0 mm
- net +5V: track 221.7 -> 239.6 mm
- net MOSI: track 81.5 -> 64.6 mm
- net MISO: track 50.8 -> 67.3 mm
- net SCK: track 66.8 -> 81.2 mm
- net N$4: track 122.0 -> 113.0 mm
- net N$11: track 0.00 -> 6.01 mm
- net N$13: track 18.7 -> 14.7 mm
- net RST: track 99.2 -> 96.6 mm, vias 1 -> 0
- net GND: vias 69 -> 66
Other:
- board text added: "044"
- board text removed: "027"
