File: pcb/Radio_bridge.sch (EAGLE design)
At the start: 45 parts, among them IC1 LM833D, J1 SJ-2509N, J2 SJ1-3523N, J4 G-1005B, SW1 EVQ-PF008K, SW2 EVQ-PF008K, U1 ESP32-DEVKITC-32D, U3 LMV7219M5X

Commit message: Rev2 PCB fixes
Parts:
- added C12: 100uF, ruark2:1210_CAPACITOR
Connections:
- new net N$11: C12.2, R16.3
- net GND: now also C12.1; no longer R16.3
- net MOSI: now also U1.IO23; no longer U1.IO27
- net N$4: now also U1.IO17; no longer U1.IO2
- net SCK: now also U1.IO18; no longer U1.IO5
- net SS: now also U1.IO5; no longer U1.IO18
Other:
- moved on the sheet: IC1B
Changed lines of the file:
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@@
 <part name="R16" library="ruark2" deviceset="PTV09A-4025F-A103" device="" value="10k"/>
 <part name="GND16" library="supply1" library_urn="urn:adsk.eagle:library:371" deviceset="GND" device=""/>
-<part name="GND17" library="supply1" library_urn="urn:adsk.eagle:library:371" deviceset="GND" device=""/>
 <part name="R17" library="ruark2" deviceset="0603_RESISTOR" device="" value="100"/>
 <part name="C4" library="ruark2" deviceset="0603_CAPACITOR" device="" value="100pF"/>
@@
 <part name="GND27" library="supply1" library_urn="urn:adsk.eagle:library:371" deviceset="GND" device=""/>
 <part name="P+6" library="supply1" library_urn="urn:adsk.eagle:library:371" deviceset="+5V" device=""/>
+<part name="C12" library="ruark2" deviceset="1210_CAPACITOR" device="" value="100uF"/>
+<part name="GND17" library="supply1" library_urn="urn:adsk.eagle:library:371" deviceset="GND" device=""/>
 </parts>
 <sheets>
@@
 <attribute name="VALUE" x="368.3" y="182.88" size="1.778" layer="96"/>
 </instance>
-<instance part="IC1" gate="B" x="365.76" y="142.24" smashed="yes">
-<attribute name="NAME" x="368.3" y="145.415" size="1.778" layer="95"/>
-<attribute name="VALUE" x="368.3" y="137.16" size="1.778" layer="96"/>
+<instance part="IC1" gate="B" x="330.2" y="142.24" smashed="yes">
+<attribute name="NAME" x="332.74" y="145.415" size="1.778" layer="95"/>
+<attribute name="VALUE" x="332.74" y="137.16" size="1.778" layer="96"/>
 </instance>
 <instance part="IC1" gate="P" x="365.76" y="187.96" smashed="yes"/>
-<instance part="GND15" gate="1" x="355.6" y="134.62" smashed="yes">
-<attribute name="VALUE" x="353.06" y="132.08" size="1.778" layer="96"/>
+<instance part="GND15" gate="1" x="320.04" y="134.62" smashed="yes">
+<attribute name="VALUE" x="317.5" y="132.08" size="1.778" layer="96"/>
 </instance>
 <instance part="C3" gate="G$1" x="398.78" y="187.96" smashed="yes" rot="R90">
@@
 <attribute name="VALUE" x="345.44" y="172.72" size="1.778" layer="96"/>
 </instance>
-<instance part="GND17" gate="1" x="378.46" y="157.48" smashed="yes">
-<attribute name="VALUE" x="375.92" y="154.94" size="1.778" layer="96"/>
-</instance>
 <instance part="R17" gate="G$1" x="340.36" y="190.5" smashed="yes">
 <attribute name="NAME" x="336.55" y="191.9986" size="1.778" layer="95"/>
@@
 <instance part="P+6" gate="1" x="210.82" y="81.28" smashed="yes">
 <attribute name="VALUE" x="208.28" y="76.2" size="1.778" layer="96" rot="R90"/>
+</instance>
+<instance part="C12" gate="G$1" x="378.46" y="152.4" smashed="yes" rot="R180">
+<attribute name="NAME" x="376.936" y="149.479" size="1.778" layer="95" rot="R180"/>
+<attribute name="VALUE" x="376.936" y="154.559" size="1.778" layer="96" rot="R180"/>
+</instance>
+<instance part="GND17" gate="1" x="378.46" y="142.24" smashed="yes">
+<attribute name="VALUE" x="375.92" y="139.7" size="1.778" layer="96"/>
 </instance>
 </instances>
@@
 <segment>
 <pinref part="IC1" gate="B" pin="-IN"/>
-<wire x1="358.14" y1="139.7" x2="355.6" y2="139.7" width="0.1524" layer="91"/>
-<wire x1="355.6" y1="139.7" x2="355.6" y2="137.16" width="0.1524" layer="91"/>
+<wire x1="322.58" y1="139.7" x2="320.04" y2="139.7" width="0.1524" layer="91"/>
+<wire x1="320.04" y1="139.7" x2="320.04" y2="137.16" width="0.1524" layer="91"/>
 <pinref part="GND15" gate="1" pin="GND"/>
-</segment>
-<segment>
-<pinref part="R16" gate="G$1" pin="3"/>
-<pinref part="GND17" gate="1" pin="GND"/>
 </segment>
 <segment>
@@
 <pinref part="GND27" gate="1" pin="GND"/>
 <wire x1="276.86" y1="167.64" x2="276.86" y2="165.1" width="0.1524" layer="91"/>
+</segment>
+<segment>
+<pinref part="GND17" gate="1" pin="GND"/>
+<pinref part="C12" gate="G$1" pin="1"/>
+<wire x1="378.46" y1="144.78" x2="378.46" y2="147.32" width="0.1524" layer="91"/>
 </segment>
 </net>
@@
 </segment>
 <segment>
-<pinref part="U1" gate="G$1" pin="IO27"/>
-<wire x1="109.22" y1="177.8" x2="99.06" y2="177.8" width="0.1524" layer="91"/>
-<label x="99.06" y="177.8" size="1.016" layer="95" rot="R180" xref="yes"/>
+<pinref part="U1" gate="G$1" pin="IO23"/>
+<wire x1="149.86" y1="200.66" x2="160.02" y2="200.66" width="0.1524" layer="91"/>
+<label x="160.02" y="200.66" size="1.016" layer="95" xref="yes"/>
 </segment>
 </net>
@@
 </segment>
 <segment>
+<pinref part="U1" gate="G$1" pin="IO18"/>
+<wire x1="149.86" y1="182.88" x2="160.02" y2="182.88" width="0.1524" layer="91"/>
+<label x="160.02" y="182.88" size="1.016" layer="95" xref="yes"/>
+</segment>
+</net>
+<net name="SS" class="0">
+<segment>
+<wire x1="360.68" y1="53.34" x2="347.98" y2="53.34" width="0.1524" layer="91"/>
+<label x="347.98" y="53.34" size="1.016" layer="95" rot="R180" xref="yes"/>
+<pinref part="JP2" gate="A" pin="11"/>
+</segment>
+<segment>
 <pinref part="U1" gate="G$1" pin="IO5"/>
 <wire x1="149.86" y1="180.34" x2="160.02" y2="180.34" width="0.1524" layer="91"/>
 <label x="160.02" y="180.34" size="1.016" layer="95" xref="yes"/>
-</segment>
-</net>
-<net name="SS" class="0">
-<segment>
-<wire x1="360.68" y1="53.34" x2="347.98" y2="53.34" width="0.1524" layer="91"/>
-<label x="347.98" y="53.34" size="1.016" layer="95" rot="R180" xref="yes"/>
-<pinref part="JP2" gate="A" pin="11"/>
-</segment>
-<segment>
-<pinref part="U1" gate="G$1" pin="IO18"/>
-<wire x1="149.86" y1="182.88" x2="160.02" y2="182.88" width="0.1524" layer="91"/>
-<label x="160.02" y="182.88" size="1.016" layer="95" xref="yes"/>
 </segment>
 </net>
@@
 <wire x1="200.66" y1="185.42" x2="200.66" y2="175.26" width="0.1524" layer="91"/>
 <wire x1="200.66" y1="175.26" x2="187.96" y2="175.26" width="0.1524" layer="91"/>
-<pinref part="U1" gate="G$1" pin="IO2"/>
-<wire x1="149.86" y1="167.64" x2="200.66" y2="167.64" width="0.1524" layer="91"/>
 <wire x1="200.66" y1="167.64" x2="200.66" y2="175.26" width="0.1524" layer="91"/>
 <junction x="200.66" y="175.26"/>
+<wire x1="200.66" y1="167.64" x2="172.72" y2="167.64" width="0.1524" layer="91"/>
+<pinref part="U1" gate="G$1" pin="IO17"/>
+<wire x1="172.72" y1="167.64" x2="172.72" y2="177.8" width="0.1524" layer="91"/>
+<wire x1="172.72" y1="177.8" x2="149.86" y2="177.8" width="0.1524" layer="91"/>
 </segment>
 </net>
@@
 <segment>
 <pinref part="IC1" gate="B" pin="+IN"/>
-<wire x1="355.6" y1="144.78" x2="358.14" y2="144.78" width="0.1524" layer="91"/>
-<wire x1="355.6" y1="144.78" x2="355.6" y2="149.86" width="0.1524" layer="91"/>
-<wire x1="355.6" y1="149.86" x2="381" y2="149.86" width="0.1524" layer="91"/>
-<wire x1="381" y1="149.86" x2="381" y2="142.24" width="0.1524" layer="91"/>
+<wire x1="320.04" y1="144.78" x2="322.58" y2="144.78" width="0.1524" layer="91"/>
+<wire x1="320.04" y1="144.78" x2="320.04" y2="149.86" width="0.1524" layer="91"/>
+<wire x1="320.04" y1="149.86" x2="345.44" y2="149.86" width="0.1524" layer="91"/>
+<wire x1="345.44" y1="149.86" x2="345.44" y2="142.24" width="0.1524" layer="91"/>
 <pinref part="IC1" gate="B" pin="OUT"/>
-<wire x1="381" y1="142.24" x2="373.38" y2="142.24" width="0.1524" layer="91"/>
+<wire x1="345.44" y1="142.24" x2="337.82" y2="142.24" width="0.1524" layer="91"/>
 </segment>
 </net>
@@
 </segment>
 </net>
+<net name="N$11" class="0">
+<segment>
+<pinref part="C12" gate="G$1" pin="2"/>
+<pinref part="R16" gate="G$1" pin="3"/>
+<wire x1="378.46" y1="154.94" x2="378.46" y2="160.02" width="0.1524" layer="91"/>
+</segment>
+</net>
